Commit message: restructure

File: franka_robotiq_description/urdf/robot.urdf.xacro (robot description, xacro)
@@ -27,5 +27,5 @@
   <xacro:if value="$(arg robotiq_gripper)">
     <xacro:include filename="$(find robotiq_description)/urdf/robotiq_gripper_macro.urdf.xacro"/>
-    <xacro:robotiq_gripper name="RobotiqGripperHardwareInterface" prefix="" parent="$(arg arm_id)_link8" use_fake_hardware="$(arg use_fake_hardware)">
+    <xacro:robotiq_gripper name="RobotiqGripperHardwareInterface" prefix="" parent="$(arg arm_id)_link8" use_fake_hardware="$(arg use_fake_hardware)" fake_sensor_commands="$(arg fake_sensor_commands)">
 	<origin xyz="0 0 0" rpy="0 0 ${radians(0)}" />
     </xacro:robotiq_gripper>

File: franka_robotiq_moveit_config/config/robotiq_gripper.xacro (robot description, xacro)
@@ -18,10 +18,11 @@
 	    <joint name="robotiq_85_right_finger_tip_joint" />
         </group>
-        <xacro:macro name="configure_robotiq_collisions" params="link enabled:=${[]}">
-            <!-- Disable collision checking between normal links, as these are handled by "sc" links -->
+	<xacro:property name="robotiq_links" value="${['base_link', 'left_knuckle_link', 'right_knuckle_link', 'left_finger_link', 'right_finger_link', 'left_inner_knuckle_link', 'right_inner_knuckle_link', 'left_finger_tip_link', 'right_finger_tip_link']}" />
+	<xacro:macro name="configure_robotiq_collisions" params="link enabled:=${[]}">
 	    <xacro:property name="panda_link_fmt" value="$(arg arm_id)_link{}" />
 	    <xacro:property name="robotiq_link_fmt" value="robotiq_85_{}" />
             <xacro:disable_collisions_for link="${robotiq_link_fmt.format(link)}" others="${[panda_link_fmt.format(i) for i in python.range(8)]}" />
-            <xacro:enable_collisions_for link="${robotiq_link_fmt.format(link)}" others="${[panda_link_fmt.format(i) for i in enabled]}" />
+	    <xacro:disable_collisions_for link="${robotiq_link_fmt.format(link)}" others="${[robotiq_link_fmt.format(l) for l in robotiq_links if l!=link]}" />
+	    <xacro:enable_collisions_for link="${robotiq_link_fmt.format(link)}" others="${[panda_link_fmt.format(i) for i in enabled]}" />
         </xacro:macro>
         <xacro:configure_robotiq_collisions link="base_link" enabled="${[0,1,2,3]}"/>
